Commit message: add gen2 stl file

File: happymimi_description/robots/happymimi.urdf (robot description, URDF)
Before this commit: robot megarover20, 14 links, 13 joints
Links:
- added link doutai_link; visual mesh filename=package://happymimi_description/meshes/stl/gen2_body.stl scale=0.01 0.01 0.01
Joints:
- added joint doutai_joint: type fixed, parent base_footprint, child doutai_link, origin xyz=0 0 0

File: happymimi_description/urdf/body/body.urdf.xacro (robot description, xacro)
@@ -14,4 +14,17 @@
 				</geometry>
 			</visual>
+	  </link>
+    <joint name="doutai_joint" type="fixed">
+    <xacro:insert_block name="joint_origin"/>
+    <parent link="${parent}"/>
+    <child  link="doutai_link"/>
+		</joint>
+    <link name="doutai_link">
+			<visual>
+				<origin xyz="0 0 0"/>
+				<geometry>
+          <mesh filename="package://happymimi_description/meshes/stl/gen2_body.stl" scale="0.01 0.01 0.01" />
+				</geometry>
+			</visual>
 		</link>
 	</xacro:macro>

Commit message: add stl file

File: happymimi_description/robots/happymimi.urdf (robot description, URDF)
Before this commit: robot megarover20, 15 links, 14 joints
Links:
- removed link doutai_link
Joints:
- removed joint doutai_joint

File: happymimi_description/urdf/body/body.urdf.xacro (robot description, xacro)
@@ -15,17 +15,19 @@
 			</visual>
 	  </link>
-    <joint name="doutai_joint" type="fixed">
-    <xacro:insert_block name="joint_origin"/>
-    <parent link="${parent}"/>
-    <child  link="doutai_link"/>
-		</joint>
-    <link name="doutai_link">
-			<visual>
-				<origin xyz="0 0 0"/>
-				<geometry>
-          <mesh filename="package://happymimi_description/meshes/stl/gen2_body.stl" scale="0.01 0.01 0.01" />
-				</geometry>
-			</visual>
-		</link>
+    <!--  -->
+    <!-- <joint name="doutai_joint" type="fixed"> -->
+    <!-- <xacro:insert_block name="joint_origin"/> -->
+    <!-- <parent link="${parent}"/> -->
+    <!-- <child  link="doutai_link"/> -->
+		<!-- </joint> -->
+    <!-- <link name="doutai_link"> -->
+		<!-- 	<visual> -->
+		<!-- 		<origin xyz="0 0 0"/> -->
+		<!-- 		<geometry> -->
+    <!--       <mesh filename="package://happymimi_description/meshes/stl/gen2_body.stl" scale="0.01 0.01 0.01" /> -->
+		<!-- 		</geometry> -->
+		<!-- 	</visual> -->
+		<!-- </link> -->
+    <!--  -->
 	</xacro:macro>
 </robot>

Commit message: add spine

File: happymimi_description/robots/happymimi.urdf (robot description, URDF)
Before this commit: robot megarover20, 14 links, 13 joints
Links:
- added link neck_link; visual cylinder length=0.05 radius=0.03
- added link spine_link; visual mesh filename=package://happymimi_description/meshes/stl/gen2_body.stl scale=0.01 0.01 0.01
- link base_laser_link: geometry visual mesh filename=package://happymimi_description/meshes/stl/lrf.stl
Joints:
- added joint neck_joint: type fixed, parent spine_link, child neck_link, origin xyz=0 0 0.72 rpy=0 0 0
- added joint spine_joint: type fixed, parent base_link, child spine_link, origin xyz=-0.052 0 0.166 rpy=0 0 0
- joint camera_joint: origin xyz=0 0 0.7 -> xyz=0.02 0 0.70
- joint respeaker_link_joint: origin xyz=-0.05 0 0.72 rpy=0 0 0 -> xyz=-0.05 0 0.05 rpy=0 0 0; parent base_link -> neck_link

File: happymimi_description/robots/happymimi.urdf.xacro (robot description, xacro)
@@ -1,4 +1,4 @@
 <?xml version="1.0"?>
-<robot name="megarover20" xmlns:xacro="http://ros.org/wiki/xacro">
+<robot name="happymimiGen2" xmlns:xacro="http://ros.org/wiki/xacro">
   <xacro:include filename="$(find happymimi_description)/urdf/body/body.urdf.xacro"/>
   <xacro:include filename="$(find happymimi_description)/urdf/camera/d435.urdf.xacro"/>
@@ -11,10 +11,32 @@
   </material>
   <material name="gray">
-    <color rgba="0.2 0.2 0.2 1" />
+    <color rgba="0.25 0.25 0.25 1" />
   </material>
-  <!--  lidar  -->
-  <link name="base_laser_link">
+  <!-- spine背骨 -->
+  <joint name="spine_joint" type="fixed">
+    <parent link="base_link"/>
+    <child  link="spine_link"/>
+    <origin xyz="-0.052 0 0.166" rpy="0 0 0"/>
+  </joint>
+  <link name="spine_link">
     <visual>
-      <origin xyz="0 0 -0.08" />
+      <!-- <origin xyz="&#45;0.08 0.10455 0.33" rpy="0 3.14 1.57"/> -->
+      <origin xyz="-0.05 0.10455 0.16" rpy="0 3.14 1.57"/>
+      <geometry>
+        <mesh filename="package://happymimi_description/meshes/stl/gen2_body.stl" scale="0.01 0.01 0.01" />
+      </geometry>
+      <material name="gray" />
+    </visual>
+  </link>
+  <!-- neck -->
+  <joint name="neck_joint" type="fixed">
+    <parent link="spine_link"/>
+    <child  link="neck_link"/>
+    <origin xyz="0 0 0.72" rpy="0 0 0"/>
+  </joint>
+  <link name="neck_link">
+    <visual>
+      <!-- <origin xyz="&#45;0.08 0.10455 0.33" rpy="0 3.14 1.57"/> -->
+      <origin xyz="0 0 0" rpy="0 0 0"/>
       <geometry>
         <cylinder length="0.05" radius="0.03" />
@@ -23,4 +45,5 @@
     </visual>
   </link>
+  <!--  lidar  -->
   <joint name="base_laser_link_joint" type="fixed">
     <parent link="base_link" />
@@ -28,9 +51,25 @@
     <origin xyz="0.1 0 0.06" rpy="3.14159 0.0 0.0"/>
   </joint>
+  <link name="base_laser_link">
+    <visual>
+      <!-- <origin xyz="0 0 &#45;0.08" /> -->
+      <origin xyz="0 0 -0.045" rpy="0 3.14 3.14"/>
+      <geometry>
+        <mesh filename="package://happymimi_description/meshes/stl/lrf.stl" />
+        <!-- <cylinder length="0.05" radius="0.03" /> -->
+      </geometry>
+      <material name="orange" />
+    </visual>
+  </link>
   <!--  realsense  -->
   <xacro:sensor_d435 parent="base_link">
-    <origin xyz="0 0 0.7"/>
+    <origin xyz="0.02 0 0.70"/>
   </xacro:sensor_d435>
   <!--  respeaker  -->
+  <joint name="respeaker_link_joint" type="fixed">
+    <parent link="neck_link" />
+    <child link="respeaker_link" />
+    <origin xyz="-0.05 0 0.05" rpy="0 0 0"/>
+  </joint>
   <link name="respeaker_link">
     <visual>
@@ -42,8 +81,3 @@
     </visual>
   </link>
-  <joint name="respeaker_link_joint" type="fixed">
-    <parent link="base_link" />
-    <child link="respeaker_link" />
-    <origin xyz="-0.05 0 0.72" rpy="0 0 0"/>
-  </joint>
 </robot>

File: happymimi_description/urdf/body/body.urdf.xacro (robot description, xacro)
@@ -15,13 +15,13 @@
 			</visual>
 	  </link>
-    <!--  -->
     <!-- <joint name="doutai_joint" type="fixed"> -->
     <!-- <xacro:insert_block name="joint_origin"/> -->
-    <!-- <parent link="${parent}"/> -->
+    <!-- <parent link="base_link"/> -->
     <!-- <child  link="doutai_link"/> -->
 		<!-- </joint> -->
     <!-- <link name="doutai_link"> -->
 		<!-- 	<visual> -->
-		<!-- 		<origin xyz="0 0 0"/> -->
+		<!-- 		<origin xyz="&#45;0.08 0.10455 0.33" rpy="0 3.14 1.57"/> -->
+    <!--     <color rgba="46 43 44 0.2" /> -->
 		<!-- 		<geometry> -->
     <!--       <mesh filename="package://happymimi_description/meshes/stl/gen2_body.stl" scale="0.01 0.01 0.01" /> -->
@@ -29,5 +29,4 @@
 		<!-- 	</visual> -->
 		<!-- </link> -->
-    <!--  -->
 	</xacro:macro>
 </robot>

Commit message: add happymimi_params

File: happymimi_description/robots/happymimi.urdf (robot description, URDF)
Before this commit: robot happymimiGen2, 16 links, 15 joints
Links:
- link neck_link: geometry visual cylinder length=0.03 radius=0.03
Joints:
- joint neck_joint: origin xyz=0 0 0.72 rpy=0 0 0 -> xyz=0 0 0.75 rpy=0 0 0

File: happymimi_description/robots/happymimi.urdf.xacro (robot description, xacro)
@@ -13,5 +13,5 @@
     <color rgba="0.25 0.25 0.25 1" />
   </material>
-  <!-- spine背骨 -->
+  <!-- spine -->
   <joint name="spine_joint" type="fixed">
     <parent link="base_link"/>
@@ -21,5 +21,4 @@
   <link name="spine_link">
     <visual>
-      <!-- <origin xyz="&#45;0.08 0.10455 0.33" rpy="0 3.14 1.57"/> -->
       <origin xyz="-0.05 0.10455 0.16" rpy="0 3.14 1.57"/>
       <geometry>
@@ -30,15 +29,16 @@
   </link>
   <!-- neck -->
-  <joint name="neck_joint" type="fixed">
-    <parent link="spine_link"/>
-    <child  link="neck_link"/>
-    <origin xyz="0 0 0.72" rpy="0 0 0"/>
+  <joint name="neck_joint" type="revolute">
+    <parent link="spine_link" />
+    <child  link="neck_link" />
+    <origin xyz="0 0 0.75" rpy="0 0 0" />
+    <axis xyz="0 1 0" />
+    <limit lower="-1.5" upper="1.5" effort="1000" velocity="0.5" />
   </joint>
   <link name="neck_link">
     <visual>
-      <!-- <origin xyz="&#45;0.08 0.10455 0.33" rpy="0 3.14 1.57"/> -->
       <origin xyz="0 0 0" rpy="0 0 0"/>
       <geometry>
-        <cylinder length="0.05" radius="0.03" />
+        <cylinder length="0.03" radius="0.03" />
       </geometry>
       <material name="gray" />

Commit message: Fix:spine_linkを円柱に修正

File: happymimi_description/robots/happymimi.urdf (robot description, URDF)
Before this commit: robot happymimiGen2, 16 links, 15 joints
Links:
- link spine_link: geometry visual cylinder length=0.722 radius=0.02
Joints:
- joint neck_joint: axis (none) -> 0 1 0; limit (none) -> lower=-1.5 upper=1.5 effort=1000 velocity=0.5; origin xyz=0 0 0.75 rpy=0 0 0 -> xyz=0 0 0.722 rpy=0 0 0; type fixed -> revolute
- joint spine_joint: origin xyz=-0.052 0 0.166 rpy=0 0 0 -> xyz=-0.03 0 0.165 rpy=0 0 0

File: happymimi_description/robots/happymimi.urdf.xacro (robot description, xacro)
@@ -17,11 +17,11 @@
     <parent link="base_link"/>
     <child  link="spine_link"/>
-    <origin xyz="-0.052 0 0.166" rpy="0 0 0"/>
+    <origin xyz="-0.03 0 0.165" rpy="0 0 0"/>
   </joint>
   <link name="spine_link">
     <visual>
-      <origin xyz="-0.05 0.10455 0.16" rpy="0 3.14 1.57"/>
+      <origin xyz="0 0 0.361" rpy="0 0 0"/>
       <geometry>
-        <mesh filename="package://happymimi_description/meshes/stl/gen2_body.stl" scale="0.01 0.01 0.01" />
+        <cylinder length="0.722" radius="0.02" />
       </geometry>
       <material name="gray" />
@@ -32,5 +32,5 @@
     <parent link="spine_link" />
     <child  link="neck_link" />
-    <origin xyz="0 0 0.75" rpy="0 0 0" />
+    <origin xyz="0 0 0.722" rpy="0 0 0" />
     <axis xyz="0 1 0" />
     <limit lower="-1.5" upper="1.5" effort="1000" velocity="0.5" />

Commit message: Fix:xacroファイルの軽微な修正

File: happymimi_description/robots/happymimi.urdf (robot description, URDF)
Before this commit: robot happymimiGen2, 16 links, 15 joints
Joints:
- joint base_laser_link_joint: origin xyz=0.1 0 0.06 rpy=3.14159 0.0 0.0 -> xyz=0.1 0 0.105 rpy=3.14159 0.0 0.0
- joint camera_joint: origin xyz=0.02 0 0.70 -> xyz=0.07 0 0.15; parent base_link -> neck_link
- joint respeaker_link_joint: origin xyz=-0.05 0 0.05 rpy=0 0 0 -> xyz=0 0 0.2 rpy=0 0 0

File: happymimi_description/robots/happymimi.urdf.xacro (robot description, xacro)
@@ -30,4 +30,5 @@
   <!-- neck -->
   <joint name="neck_joint" type="revolute">
+  <!-- <joint name="neck_joint" type="fixed"> -->
     <parent link="spine_link" />
     <child  link="neck_link" />
@@ -49,13 +50,11 @@
     <parent link="base_link" />
     <child link="base_laser_link" />
-    <origin xyz="0.1 0 0.06" rpy="3.14159 0.0 0.0"/>
+    <origin xyz="0.1 0 0.105" rpy="3.14159 0.0 0.0"/>
   </joint>
   <link name="base_laser_link">
     <visual>
-      <!-- <origin xyz="0 0 &#45;0.08" /> -->
-      <origin xyz="0 0 -0.045" rpy="0 3.14 3.14"/>
+      <origin xyz="0 0 0" rpy="0 3.14 3.14"/>
       <geometry>
         <mesh filename="package://happymimi_description/meshes/stl/lrf.stl" />
-        <!-- <cylinder length="0.05" radius="0.03" /> -->
       </geometry>
       <material name="orange" />
@@ -63,6 +62,6 @@
   </link>
   <!--  realsense  -->
-  <xacro:sensor_d435 parent="base_link">
-    <origin xyz="0.02 0 0.70"/>
+  <xacro:sensor_d435 parent="neck_link">
+    <origin xyz="0.07 0 0.15"/>
   </xacro:sensor_d435>
   <!--  respeaker  -->
@@ -70,5 +69,5 @@
     <parent link="neck_link" />
     <child link="respeaker_link" />
-    <origin xyz="-0.05 0 0.05" rpy="0 0 0"/>
+    <origin xyz="0 0 0.2" rpy="0 0 0"/>
   </joint>
   <link name="respeaker_link">

File: happymimi_description/urdf/body/body.urdf.xacro (robot description, xacro)
@@ -15,18 +15,4 @@
 			</visual>
 	  </link>
-    <!-- <joint name="doutai_joint" type="fixed"> -->
-    <!-- <xacro:insert_block name="joint_origin"/> -->
-    <!-- <parent link="base_link"/> -->
-    <!-- <child  link="doutai_link"/> -->
-		<!-- </joint> -->
-    <!-- <link name="doutai_link"> -->
-		<!-- 	<visual> -->
-		<!-- 		<origin xyz="&#45;0.08 0.10455 0.33" rpy="0 3.14 1.57"/> -->
-    <!--     <color rgba="46 43 44 0.2" /> -->
-		<!-- 		<geometry> -->
-    <!--       <mesh filename="package://happymimi_description/meshes/stl/gen2_body.stl" scale="0.01 0.01 0.01" /> -->
-		<!-- 		</geometry> -->
-		<!-- 	</visual> -->
-		<!-- </link> -->
 	</xacro:macro>
 </robot>

Commit message: Fix: 2dlidar.launchファイルを修正

File: happymimi_description/robots/happymimi.urdf (robot description, URDF)
Before this commit: robot happymimiGen2, 16 links, 15 joints
Joints:
- joint base_laser_link_joint: parent base_link -> base_footprint

File: happymimi_description/robots/happymimi.urdf.xacro (robot description, xacro)
@@ -48,5 +48,5 @@
   <!--  lidar  -->
   <joint name="base_laser_link_joint" type="fixed">
-    <parent link="base_link" />
+    <parent link="base_footprint" />
     <child link="base_laser_link" />
     <origin xyz="0.1 0 0.105" rpy="3.14159 0.0 0.0"/>
@@ -57,4 +57,5 @@
       <geometry>
         <mesh filename="package://happymimi_description/meshes/stl/lrf.stl" />
+        <!-- <cylinder length="0.09" radius="0.03" /> -->
       </geometry>
       <material name="orange" />
@@ -62,6 +63,8 @@
   </link>
   <!--  realsense  -->
-  <xacro:sensor_d435 parent="neck_link">
-    <origin xyz="0.07 0 0.15"/>
+  <!-- <xacro:sensor_d435 parent="neck_link"> -->
+  <xacro:sensor_d435 parent="base_link">
+    <!-- <origin xyz="0.07 0 0.15"/> -->
+    <origin xyz="0.01 0 0.8"/>
   </xacro:sensor_d435>
   <!--  respeaker  -->
