Commit message: Fix: ロボットモデルの修正

File: happymimi_description/robots/happymimi.urdf.xacro (robot description, xacro)
@@ -23,5 +23,5 @@
       <origin xyz="0 0 0.361" rpy="0 0 0"/>
       <geometry>
-        <cylinder length="0.722" radius="0.02" />
+        <box size="0.03 0.03 0.72"/>
       </geometry>
       <material name="gray" />
@@ -41,5 +41,6 @@
       <origin xyz="0 0 0" rpy="0 0 0"/>
       <geometry>
-        <cylinder length="0.03" radius="0.03" />
+        <!-- <cylinder length="0.03" radius="0.03" /> -->
+        <box size="0.05 0.045 0.09 " />
       </geometry>
       <material name="gray" />
@@ -63,8 +64,8 @@
   </link>
   <!--  realsense  -->
-  <!-- <xacro:sensor_d435 parent="neck_link"> -->
-  <xacro:sensor_d435 parent="base_link">
-    <!-- <origin xyz="0.07 0 0.15"/> -->
-    <origin xyz="0.01 0 0.8"/>
+  <xacro:sensor_d435 parent="neck_link">
+  <!-- <xacro:sensor_d435 parent="base_link"> -->
+    <origin xyz="0.07 0 0.15"/>
+    <!-- <origin xyz="0.01 0 0.8"/> -->
   </xacro:sensor_d435>
   <!--  respeaker  -->

Commit message: Fix: d435iに対応

File: happymimi_description/robots/happymimi.urdf.xacro (robot description, xacro)
@@ -2,5 +2,6 @@
 <robot name="happymimiGen2" xmlns:xacro="http://ros.org/wiki/xacro">
   <xacro:include filename="$(find happymimi_description)/urdf/body/body.urdf.xacro"/>
-  <xacro:include filename="$(find happymimi_description)/urdf/camera/d435.urdf.xacro"/>
+  <!-- <xacro:include filename="$(find happymimi_description)/urdf/camera/d435.urdf.xacro"/> -->
+  <xacro:include filename="$(find realsense2_description)/urdf/_d435i.urdf.xacro"/>
   <link name="base_footprint"/>
   <xacro:body parent="base_footprint">
@@ -64,9 +65,12 @@
   </link>
   <!--  realsense  -->
-  <xacro:sensor_d435 parent="neck_link">
-  <!-- <xacro:sensor_d435 parent="base_link"> -->
-    <origin xyz="0.07 0 0.15"/>
-    <!-- <origin xyz="0.01 0 0.8"/> -->
-  </xacro:sensor_d435>
+  <!-- <xacro:sensor_d435 parent="neck_link"> -->
+  <!-- <!-1- <xacro:sensor_d435 parent="base_link"> -1-> -->
+  <!--   <origin xyz="0.07 0 0.15"/> -->
+  <!--   <!-1- <origin xyz="0.01 0 0.8"/> -1-> -->
+  <!-- </xacro:sensor_d435> -->
+  <xacro:sensor_d435i parent="base_link" use_nominal_extrinsics="false">
+    <origin xyz="0 0 0.90"/>
+  </xacro:sensor_d435i>
   <!--  respeaker  -->
   <joint name="respeaker_link_joint" type="fixed">

Commit message: aaaaaa

File: happymimi_description/robots/happymimi.urdf.xacro (robot description, xacro)
@@ -70,6 +70,8 @@
   <!--   <!-1- <origin xyz="0.01 0 0.8"/> -1-> -->
   <!-- </xacro:sensor_d435> -->
-  <xacro:sensor_d435i parent="base_link" use_nominal_extrinsics="false">
-    <origin xyz="0 0 0.90"/>
+  <!-- <xacro:sensor_d435i parent="base_link" use_nominal_extrinsics="false"> -->
+  <xacro:sensor_d435i parent="neck_link" use_nominal_extrinsics="false">
+    <!-- <origin xyz="0 0 0.90"/> -->
+    <origin xyz="0.07 0 0.15"/>
   </xacro:sensor_d435i>
   <!--  respeaker  -->

Commit message: Fix: りあるせんすのリンクを修正

File: happymimi_description/robots/happymimi.urdf.xacro (robot description, xacro)
@@ -70,8 +70,8 @@
   <!--   <!-1- <origin xyz="0.01 0 0.8"/> -1-> -->
   <!-- </xacro:sensor_d435> -->
-  <!-- <xacro:sensor_d435i parent="base_link" use_nominal_extrinsics="false"> -->
-  <xacro:sensor_d435i parent="neck_link" use_nominal_extrinsics="false">
-    <!-- <origin xyz="0 0 0.90"/> -->
-    <origin xyz="0.07 0 0.15"/>
+  <xacro:sensor_d435i parent="base_link" use_nominal_extrinsics="false">
+  <!-- <xacro:sensor_d435i parent="neck_link" use_nominal_extrinsics="false"> -->
+    <origin xyz="0 0 0.90"/>
+    <!-- <origin xyz="0.07 0 0.15"/> -->
   </xacro:sensor_d435i>
   <!--  respeaker  -->

Commit message: Fix: realsenseの座標を修正:wq

File: happymimi_description/robots/happymimi.urdf.xacro (robot description, xacro)
@@ -70,8 +70,8 @@
   <!--   <!-1- <origin xyz="0.01 0 0.8"/> -1-> -->
   <!-- </xacro:sensor_d435> -->
-  <xacro:sensor_d435i parent="base_link" use_nominal_extrinsics="false">
-  <!-- <xacro:sensor_d435i parent="neck_link" use_nominal_extrinsics="false"> -->
-    <origin xyz="0 0 0.90"/>
-    <!-- <origin xyz="0.07 0 0.15"/> -->
+  <!-- <xacro:sensor_d435i parent="base_link" use_nominal_extrinsics="false"> -->
+  <xacro:sensor_d435i parent="neck_link" use_nominal_extrinsics="false">
+    <!-- <origin xyz="0 0 0.90"/> -->
+    <origin xyz="0.07 0 0.15"/>
   </xacro:sensor_d435i>
   <!--  respeaker  -->

Commit message: Fix: 軽微な修正

File: happymimi_description/robots/happymimi.urdf.xacro (robot description, xacro)
@@ -30,5 +30,5 @@
   </link>
   <!-- neck -->
-  <joint name="neck_joint" type="revolute">
+  <joint name="m5_neck_joint" type="revolute">
   <!-- <joint name="neck_joint" type="fixed"> -->
     <parent link="spine_link" />

Commit message: Fix: 首のジョイント角度を０になるよう修正

File: happymimi_description/robots/happymimi.urdf.xacro (robot description, xacro)
@@ -1,3 +1,3 @@
-<?xml version="1.0"?>
+<?xml version="1.0" encoding="utf-8"?>
 <robot name="happymimiGen2" xmlns:xacro="http://ros.org/wiki/xacro">
   <xacro:include filename="$(find happymimi_description)/urdf/body/body.urdf.xacro"/>
@@ -34,5 +34,5 @@
     <parent link="spine_link" />
     <child  link="neck_link" />
-    <origin xyz="0 0 0.722" rpy="0 0 0" />
+    <origin xyz="0 0 0.722" rpy="0 0.38 0" />
     <axis xyz="0 1 0" />
     <limit lower="-1.5" upper="1.5" effort="1000" velocity="0.5" />

Commit message: Add: IMUとCameraの２種類のリアルセンスリンクを追加

File: happymimi_description/robots/happymimi.urdf.xacro (robot description, xacro)
@@ -2,5 +2,5 @@
 <robot name="happymimiGen2" xmlns:xacro="http://ros.org/wiki/xacro">
   <xacro:include filename="$(find happymimi_description)/urdf/body/body.urdf.xacro"/>
-  <!-- <xacro:include filename="$(find happymimi_description)/urdf/camera/d435.urdf.xacro"/> -->
+  <xacro:include filename="$(find realsense2_description)/urdf/_d435.urdf.xacro"/>
   <xacro:include filename="$(find realsense2_description)/urdf/_d435i.urdf.xacro"/>
   <link name="base_footprint"/>
@@ -64,15 +64,17 @@
     </visual>
   </link>
-  <!--  realsense  -->
-  <!-- <xacro:sensor_d435 parent="neck_link"> -->
-  <!-- <!-1- <xacro:sensor_d435 parent="base_link"> -1-> -->
-  <!--   <origin xyz="0.07 0 0.15"/> -->
-  <!--   <!-1- <origin xyz="0.01 0 0.8"/> -1-> -->
-  <!-- </xacro:sensor_d435> -->
+  <!--  realsense for IMU  -->
+  <xacro:sensor_d435i parent="base_link" use_nominal_extrinsics="false">
+    <origin xyz="0.1 0 0.085"/>
+  </xacro:sensor_d435i>
+  <!--  realsense for RGB-D Camera -->
+  <xacro:sensor_d435 parent="neck_link">
+    <origin xyz="0.07 0 0.15"/>
+  </xacro:sensor_d435>
   <!-- <xacro:sensor_d435i parent="base_link" use_nominal_extrinsics="false"> -->
-  <xacro:sensor_d435i parent="neck_link" use_nominal_extrinsics="false">
+  <!-- <xacro:sensor_d435i parent="neck_link" use_nominal_extrinsics="false"> -->
     <!-- <origin xyz="0 0 0.90"/> -->
-    <origin xyz="0.07 0 0.15"/>
-  </xacro:sensor_d435i>
+    <!-- <origin xyz="0.07 0 0.15"/> -->
+  <!-- </xacro:sensor_d435i> -->
   <!--  respeaker  -->
   <joint name="respeaker_link_joint" type="fixed">

Commit message: Fix: 軽微な修正

File: happymimi_description/robots/happymimi.urdf.xacro (robot description, xacro)
@@ -2,5 +2,5 @@
 <robot name="happymimiGen2" xmlns:xacro="http://ros.org/wiki/xacro">
   <xacro:include filename="$(find happymimi_description)/urdf/body/body.urdf.xacro"/>
-  <xacro:include filename="$(find realsense2_description)/urdf/_d435.urdf.xacro"/>
+  <!-- <xacro:include filename="$(find realsense2_description)/urdf/_d435.urdf.xacro"/> -->
   <xacro:include filename="$(find realsense2_description)/urdf/_d435i.urdf.xacro"/>
   <link name="base_footprint"/>
@@ -69,7 +69,7 @@
   </xacro:sensor_d435i>
   <!--  realsense for RGB-D Camera -->
-  <xacro:sensor_d435 parent="neck_link">
-    <origin xyz="0.07 0 0.15"/>
-  </xacro:sensor_d435>
+  <!-- <xacro:sensor_d435 parent="neck_link"> -->
+    <!-- <origin xyz="0.07 0 0.15"/> -->
+  <!-- </xacro:sensor_d435> -->
   <!-- <xacro:sensor_d435i parent="base_link" use_nominal_extrinsics="false"> -->
   <!-- <xacro:sensor_d435i parent="neck_link" use_nominal_extrinsics="false"> -->

Commit message: 2021/11/15

File: happymimi_description/robots/happymimi.urdf.xacro (robot description, xacro)
@@ -3,5 +3,5 @@
   <xacro:include filename="$(find happymimi_description)/urdf/body/body.urdf.xacro"/>
   <xacro:include filename="$(find realsense2_description)/urdf/_d435.urdf.xacro"/>
-  <xacro:include filename="$(find realsense2_description)/urdf/_d435i.urdf.xacro"/>
+  <!-- <xacro:include filename="$(find realsense2_description)/urdf/_d435i.urdf.xacro"/> -->
   <link name="base_footprint"/>
   <xacro:body parent="base_footprint">
@@ -65,7 +65,22 @@
   </link>
   <!--  realsense for IMU  -->
-  <xacro:sensor_d435i parent="base_link" use_nominal_extrinsics="false">
-    <origin xyz="0.1 0 0.085"/>
-  </xacro:sensor_d435i>
+  <!-- <xacro:sensor_d435i parent="base_link" use_nominal_extrinsics="false"> -->
+    <!-- <origin xyz="0.1 0 0.085"/> -->
+  <!-- </xacro:sensor_d435i> -->
+  <!-- IMU -->
+  <joint name="imu_joint" type="fixed">
+    <parent link="base_link" />
+    <child link="imu_link" />
+    <origin xyz="-0.03 0.05 0.185" rpy="0.0 0.0 0.0"/>
+  </joint>
+  <link name="imu_link">
+    <visual>
+      <origin xyz="0 0 0" rpy="0 0 0"/>
+      <geometry>
+        <box size="0.03 0.03 0.004"/>
+      </geometry>
+      <material name="orange" />
+    </visual>
+  </link>
   <!--  realsense for RGB-D Camera -->
   <xacro:sensor_d435 parent="neck_link">

Commit message: Fix: realsenseのコメントアウトはずす

File: happymimi_description/robots/happymimi.urdf.xacro (robot description, xacro)
@@ -48,5 +48,5 @@
     </visual>
   </link>
-  <!--  lidar  -->
+  <!--  2d-lidar  -->
   <joint name="base_laser_link_joint" type="fixed">
     <parent link="base_footprint" />
@@ -64,8 +64,4 @@
     </visual>
   </link>
-  <!--  realsense for IMU  -->
-  <!-- <xacro:sensor_d435i parent="base_link" use_nominal_extrinsics="false"> -->
-    <!-- <origin xyz="0.1 0 0.085"/> -->
-  <!-- </xacro:sensor_d435i> -->
   <!-- IMU -->
   <joint name="imu_joint" type="fixed">
@@ -84,7 +80,7 @@
   </link>
   <!--  realsense for RGB-D Camera -->
-  <!-- <xacro:sensor_d435 parent="neck_link"> -->
-    <!-- <origin xyz="0.07 0 0.15"/> -->
-  <!-- </xacro:sensor_d435> -->
+  <xacro:sensor_d435 parent="neck_link">
+    <origin xyz="0.07 0 0.15"/>
+  </xacro:sensor_d435>
   <!-- <xacro:sensor_d435i parent="base_link" use_nominal_extrinsics="false"> -->
   <!-- <xacro:sensor_d435i parent="neck_link" use_nominal_extrinsics="false"> -->
